File: forte-encoder-pcb/forte-encoder-pcb.kicad_sch (KiCad schematic)
At the start: 2 parts, among them U1 MA732GQ-P, U2 STM32F103C8Tx

Commit message: wip
Parts:
- removed U1: MA732GQ-P, QFN-16_MA732, symbol MA732:MA732GQ-P
- added C24, C28, C29, C30, C31, C35, C36: 100nF 50V, dash:CC0603JRX7R9BB104, symbol dash:CC0603JRX7R9BB104
- added C32: CL31B105KCHNNNE, dash:CL31B105KCHNNNE, symbol dash:CL31B105KCHNNNE
- added C33: 1uF 100V, dash:GRM21BC72A105KE01L, symbol dash:GRM21BC72A105KE01L
- added C37: CL31B225KCHSNNE, dash:CL31B225KCHSNNE, symbol dash:CL31B225KCHSNNE
- added C38: CL10B222KB8NNNC, dash:CL10B222KB8NNNC, symbol dash:CL10B222KB8NNNC
- added C39: GRM31CR61E476ME44L, dash:GRM31CR61E476ME44L, symbol dash:GRM31CR61E476ME44L
- added C40, C41: GRM32ER71E226KE15L, dash:GRM32ER71E226KE15L, symbol dash:GRM32ER71E226KE15L
- added C42: CC0402JRNPO9BN560, dash:RC0402FR_0752K3L, symbol Device:C
- added C43: Samsung Electro-Mechanics CL10B332KB8NNNC, dash:CC0603JRX7R9BB104, symbol Device:C
- added C54: 100nF 100V, dash:CL10B104KC8NNNC, symbol dash:CL10B104KC8NNNC
- added CN1, CN2: (no value), dash:xt-30, symbol dash:XT30PW-M
- added CN3(OUT)1, CN3(OUT)2: XT30(2+2)PB-M.G.B, dash:XT30(2+2)PB-M.G.B, symbol dash:XT30(2+2)PB-M.G.B
- added D2: LITEON LTST-C191KRKT, dash:LTST_C191KRKT, symbol dash:LTST-C191KRKT
- added FL1: BLM18AG601SN1D, dash:BLM18AG601SN1D, symbol dash:BLM18AG601SN1D
- added J1: BM07B-SRSS-TB(LF)(SN), dash:BM07B-SRSS-TB, symbol dash:BM07B-SRSS-TB
- added L1: TDK VLS5045EX-680M, dash:VLS5045EX_680M, symbol dash:VLS5045EX_680M
- added L2, L3: DFE252012PD-2R2M=P2, dash:DFE252012PD_2R2M_P2, symbol dash:DFE252012PD_2R2M_P2
- added R10: RC0402FR-0742K2L, dash:RC0402FR_0742K2L, symbol dash:RC0402FR_0742K2L
- added R11: RC0402FR-0780K6L, dash:RC0402FR_0780K6L, symbol dash:RC0402FR_0780K6L
- added R12: RC0402FR-0752K3L, dash:RC0402FR_0752K3L, symbol dash:RC0402FR_0752K3L
- added R13: RC0805FR-07100KL, dash:RC0805FR_07100KL, symbol dash:RC0805FR_07100KL
- added R14: RT0603BRD0749K9L, dash:RT0603BRD0749K9L, symbol dash:RT0603BRD0749K9L
- added R15, R9: 0603WAF4533T5E, dash:RT0603BRD07448KL, symbol Device:R
- added R8: 200oh, dash:RC0402JR-07200RL, symbol dash:RC0402JR-07200RL
- added TP1: +12V TestPoint, TestPoint:TestPoint_THTPad_D1.5mm_Drill0.7mm, symbol Connector:TestPoint
- added TP11: TP_MOSI, TestPoint:TestPoint_THTPad_D1.0mm_Drill0.5mm, symbol Connector:TestPoint
- added TP12: TP_CS, TestPoint:TestPoint_THTPad_D1.0mm_Drill0.5mm, symbol Connector:TestPoint
- added TP13: TP_MISO, TestPoint:TestPoint_THTPad_D1.0mm_Drill0.5mm, symbol Connector:TestPoint
- added TP14: TP_SCK, TestPoint:TestPoint_THTPad_D1.0mm_Drill0.5mm, symbol Connector:TestPoint
- added TP2: +48V TestPoint, TestPoint:TestPoint_THTPad_D1.5mm_Drill0.7mm, symbol Connector:TestPoint
- added TP3: +5V TestPoint, TestPoint:TestPoint_THTPad_D1.5mm_Drill0.7mm, symbol Connector:TestPoint
- added TP4: +3.3V TestPoint, TestPoint:TestPoint_THTPad_D1.5mm_Drill0.7mm, symbol Connector:TestPoint
- added TP_GND1, TP_GND2: GND TestPoint, TestPoint:TestPoint_THTPad_D1.5mm_Drill0.7mm, symbol Connector:TestPoint
- added U3: MCP2542FD-E/MF, dash:MCP2542FD_E_MF, symbol dash:MCP2542FD-E_MF
- added U4: MA732GQ-Z, dash:MA732GQ-Z, symbol dash:MA732GQ-Z
- added U5, U6: TPS629203DRLR, dash:TPS629203DRLR, symbol dash:TPS629203DRLR
- added VR1: LM5164DDAR, dash:LM5164DDAR, symbol dash:LM5164DDAR
- added Y1: CSTNE8M00G550000R0, dash:CSTNE8M00G550000R0, symbol dash:CSTNE8M00G550000R0
Connections:
- net SCK: now reaches U2.15 (PA5)
- net SCK: now also TP14.1, U4.12 (SCLK)
- net +3.3V: now reaches U2.48 (VDD)
- net +3.3V: now also U2.1 (VBAT), U2.24 (VDD), U2.36 (VDD), C28.2, C29.2, C30.2, C31.2, C32.2, C33.2, C36.1, C41.2, C54.1, FL1.1, J1.1, L3.2, TP4.1, U3.5 (VIO), U4.13 (VDD), U6.3 (VOS)
- net MOSI: now reaches U2.17 (PA7)
- net MOSI: now also TP11.1, U4.4 (MOSI)
- net CS: now reaches U2.14 (PA4)
- net CS: now also TP12.1, U4.5 (CS)
- net MISO: now reaches U2.16 (PA6)
- net MISO: now also TP13.1, U4.7 (MISO)
- net GND: now reaches U2.23 (VSS), U2.35 (VSS), U2.47 (VSS)
- net GND: now also U2.44 (BOOT0), U2.8 (VSSA), C24.2, C28.1, C29.1, C30.1, C31.1, C32.1, C33.1, C35.2, C36.2, C37.1, C39.1, C40.1, C41.1, C54.2, CN3(OUT)1.3, CN3(OUT)2.3, D2.1, J1.3, R10.1, R11.1, R12.1, R13.1, R14.1, TP_GND1.1, TP_GND2.1, U3.2 (VSS), U3.8 (STBY), U3.9 (EPAD), U4.17 (PAD), U4.8 (GND), U5.5 (GND), U6.5 (GND), VR1.1 (GND), VR1.9 (EP), Y1.2
- net USART_TX: now reaches U2.12 (PA2)
- net USART_TX: now also J1.6
- net USART_RX: now reaches U2.13 (PA3)
- net USART_RX: now also J1.7
- net CAN_RX: now reaches U2.32 (PA11)
- net CAN_RX: now also U3.4 (RXD)
- net CAN_TX: now reaches U2.33 (PA12)
- net CAN_TX: now also U3.1 (TXD)
- net TCK: now reaches U2.37 (PA14)
- net TCK: now also J1.2
- net TMS: now reaches U2.38 (PA15)
- net TMS: now also J1.4
- net INDICATOR: now reaches U2.41 (PB5)
- net INDICATOR: now also R8.1
- net RCC_OSC_IN: now reaches U2.5 (PD0)
- net RCC_OSC_IN: now also Y1.1
- net RCC_OSC_OUT: now reaches U2.6 (PD1)
- net RCC_OSC_OUT: now also Y1.3
- net NRST: now reaches U2.7 (NRST)
- net NRST: now also J1.5
- net at U2.9 (VDDA): now also C24.1, FL1.2
- new net: C38.2, L1.1, R15.1, VR1.8 (SW)
- new net: C42.1, C43.1, R15.2
- new net: C42.2, R14.2, R9.2, VR1.5 (FB)
- new net: D2.2, R8.2
- new net: R10.2, U5.8 (MODE/S-CONF)
- new net: R11.2, U5.1 (FB/VSET)
- new net: L3.1, U6.4 (SW)
- new net: R12.2, U6.8 (MODE/S-CONF)
- new net: L2.1, U5.4 (SW)
- new net: R13.2, VR1.4 (RON)
- new net: C38.1, VR1.7 (BST)
- new net +12V: C39.2, C43.2, L1.2, R9.1, TP1.1, U5.6 (VIN), U5.7 (EN)
- new net +48V: C37.2, CN3(OUT)1.4, CN3(OUT)2.4, TP2.1, VR1.2 (VIN), VR1.3 (EN/UVLO)
- new net +5V: C35.1, C40.2, L2.2, TP3.1, U3.3 (VDD), U5.3 (VOS), U6.6 (VIN), U6.7 (EN)
- new net CAN+: CN3(OUT)1.1, CN3(OUT)2.1, U3.7 (CANH)
- new net CAN-: CN3(OUT)1.2, CN3(OUT)2.2, U3.6 (CANL)
- no-connect marks 0 -> 38
Other:
- note added: "Auxiliaries"
- note added: "CAN"
- note added: "Encoder"
- note added: "MCU"
- note added: "Power"
- moved on the sheet: U2

Commit message: halp
Parts:
- removed CN1, CN2: (no value), dash:xt-30, symbol dash:XT30PW-M
- removed CN3(OUT)2: XT30(2+2)PB-M.G.B, dash:XT30(2+2)PB-M.G.B, symbol dash:XT30(2+2)PB-M.G.B
- added J10, J11, J6, J7, J8, J9: Conn_01x01_Pin, TestPoint:TestPoint_Plated_Hole_D2.0mm, symbol Connector:Conn_01x01_Pin

Commit message: modify pcb
Parts:
- renumbered J1 to J0, J7 to J1, J11 to J2, J10 to J3, J8 to J4, J6 to J5, J9 to J6
Connections:
- net +48V: now also J1.1 (Pin_1), J2.1 (Pin_1), J3.1 (Pin_1)
- net GND: now also J4.1 (Pin_1), J5.1 (Pin_1), J6.1 (Pin_1)
Other:
- moved on the sheet: J1, J3, J4, J5, J6

Commit message: super messy
Parts:
- added J10, J7, J8, J9: Conn_01x01_Pin, TestPoint:TestPoint_THTPad_D1.5mm_Drill0.7mm, symbol Connector:Conn_01x01_Pin
Connections:
- net CAN+: now also J10.1 (Pin_1), J7.1 (Pin_1)
- net CAN-: now also J8.1 (Pin_1), J9.1 (Pin_1)
