File: forte-encoder-pcb/forte-encoder-pcb.kicad_sch (KiCad schematic)
At the start: 59 parts, among them CN3(OUT)1 XT30(2+2)PB-M.G.B, J0 BM07B-SRSS-TB(LF)(SN), J1 Conn_01x01_Pin, J10 Conn_01x01_Pin, J2 Conn_01x01_Pin, J3 Conn_01x01_Pin, J4 Conn_01x01_Pin, J5 Conn_01x01_Pin, J6 Conn_01x01_Pin, J7 Conn_01x01_Pin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

Commit message: push all changes
Parts:
- removed TP2: +48V TestPoint, TestPoint:TestPoint_THTPad_D1.5mm_Drill0.7mm, symbol Connector:TestPoint
- removed TP_GND1, TP_GND2: GND TestPoint, TestPoint:TestPoint_THTPad_D1.5mm_Drill0.7mm, symbol Connector:TestPoint
- added CN1: (no value), dash:CONN-TH_XT30UPB-F, symbol dash:XT30UPB-F30.G.Y
- J1, J2, J3, J4, J5, J6: footprint TestPoint:TestPoint_Plated_Hole_D2.0mm -> TestPoint:TestPoint_Loop_D2.54mm_Drill1.5mm_Beaded
- TP1, TP3, TP4: footprint TestPoint:TestPoint_THTPad_D1.5mm_Drill0.7mm -> TestPoint:TestPoint_Pad_D1.5mm
- TP11, TP12, TP13, TP14: footprint TestPoint:TestPoint_THTPad_D1.0mm_Drill0.5mm -> TestPoint:TestPoint_Pad_D1.0mm
