File: forte-encoder-pcb/forte-encoder-pcb.kicad_pcb (KiCad board)
At the start: 6 copper layers, 36.5 x 45 mm, 62 parts, among them CN3(OUT)1 XT30(2+2)PB-M.G.B, J0 BM07B-SRSS-TB(LF)(SN), J1 Conn_01x01_Pin, J10 Conn_01x01_Pin, J2 Conn_01x01_Pin, J3 Conn_01x01_Pin, J4 Conn_01x01_Pin, J5 Conn_01x01_Pin, J6 Conn_01x01_Pin, J7 Conn_01x01_Pin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

Commit message: push all changes
Parts:
- removed REF**: MountingHole_2.1mm, MountingHole:MountingHole_2.1mm
- removed REF** (x2): MountingHole_2.2mm_M2, MountingHole:MountingHole_2.2mm_M2
- removed TP2: +48V TestPoint, TestPoint:TestPoint_THTPad_D1.5mm_Drill0.7mm
- removed TP_GND1, TP_GND2: GND TestPoint, TestPoint:TestPoint_THTPad_D1.5mm_Drill0.7mm
- added CN1: ~, dash:CONN-TH_XT30UPB-F, F.Cu at (6.53, 2.93)
- C37, R13: moved to F.Cu
- J1, J2, J3, J4, J5, J6: footprint TestPoint:TestPoint_Plated_Hole_D2.0mm -> TestPoint:TestPoint_Loop_D2.54mm_Drill1.5mm_Beaded
- R10, VR1: moved to B.Cu
- TP1, TP3, TP4: footprint TestPoint:TestPoint_THTPad_D1.5mm_Drill0.7mm -> TestPoint:TestPoint_Pad_D1.5mm
- TP11, TP12, TP13, TP14: footprint TestPoint:TestPoint_THTPad_D1.0mm_Drill0.5mm -> TestPoint:TestPoint_Pad_D1.0mm
- moved TP1 59.0 mm to (151.7, 72.7)
- moved TP4 39.2 mm to (144.1, 106.8)
- moved TP3 34.1 mm to (131.2, 69.7)
- moved J10 29.8 mm to (139.7, 96.8)
- moved CN3(OUT)1 28.9 mm to (88.7, 86.9), turned to -50 degrees
- moved R13 24.6 mm to (109.2, 84.4), turned to 140 degrees
- moved J8 22.2 mm to (131.0, 112.0)
- moved J9 22.2 mm to (133.2, 116.0)
- moved J7 22.2 mm to (135.9, 116.0)
- moved VR1 20.6 mm to (109.6, 87.4), turned to -40 degrees
- moved C38 20.3 mm to (110.9, 90.3), turned to -130 degrees
- moved R14 20.2 mm to (114.1, 90.7), turned to 140 degrees
- moved C37 19.4 mm to (108.3, 86.5), turned to 140 degrees
- moved R10 19.4 mm to (116.7, 96.0), turned to -90 degrees
- moved R9 18.1 mm to (113.2, 93.0), turned to 50 degrees
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Routing:
- net GND: track 125.7 -> 47.3 mm, vias 16 -> 65
- net +48V: track 54.8 -> 0.01 mm, vias 2 -> 56
- net +5V: track 51.4 -> 11.6 mm, vias 3 -> 2
- net +12V: track 20.5 -> 0.00 mm, vias 2 -> 0
- net +3.3V: track 56.6 -> 42.1 mm, vias 7 -> 6
- net /CAN+: track 19.8 -> 7.96 mm
- net /CAN-: track 15.5 -> 6.78 mm
- net Net-(VR1-SW): track 12.2 -> 3.67 mm, vias 1 -> 0
- net Net-(VR1-FB): track 13.2 -> 6.37 mm, vias 2 -> 0
- net Net-(VR1-BST): track 4.12 -> 0.00 mm
- net Net-(U6-SW): track 3.57 -> 0.00 mm, vias 1 -> 0
- net Net-(VR1-RON): track 2.56 -> 0.00 mm
- net Net-(C42-Pad1): track 7.19 -> 5.57 mm
- net Net-(U5-SW): track 2.73 -> 3.84 mm
- net Net-(U5-MODE/S-CONF): track 2.52 -> 1.50 mm, vias 1 -> 0
- added copper zone on B.Cu, net +48V
- added copper zone on F.Cu, net +48V
- added copper zone on In1.Cu, net +48V
- added copper zone on In3.Cu, net +48V
- added copper zone on In4.Cu, net +48V
- added copper zone on B.Cu, net GND
- added copper zone on F.Cu, net GND
- added copper zone on In2.Cu, net GND
- added copper zone on In3.Cu, net GND
